File: _3_KICAD_BASE_BOARD/dspic33ak512mps512_baseboard/BLOCK_SIGNAL_IO.kicad_sch (KiCad schematic)
At the start: 1 part, among them U1 DAC7564ICPW

Commit message: feat : 회로 작업중
Parts:
- added C26, C27, C28: 100nF, Capacitor_SMD:C_0603_1608Metric, symbol Device:C_Small
- added R4: 100R, Resistor_SMD:R_0603_1608Metric, symbol Device:R_Small
- renumbered U1 to U3
Connections:
- net DAC_0: now reaches U3.1 (VOUTA)
- net CLK: now reaches U3.10 (SCLK)
- net MOSI: now reaches U3.11 (DIN)
- net +3.3V: now reaches U3.12 (IOVDD)
- net +3.3V: now also U3.4 (AVDD), C27.1, C28.1, R4.1
- net GND: now reaches U3.13 (A0)
- net GND: now also U3.14 (A1), U3.15 (~{ENABLE}), U3.16 (LDAC), U3.5 (VREFL), U3.6 (GND), C26.2, C27.2, C28.2
- net DAC_1: now reaches U3.2 (VOUTB)
- net at U3.3 (VREFH/VREFOUT): now also C26.1, R4.2
- net DAC_2: now reaches U3.7 (VOUTC)
- net SS: now reaches U3.9 (~{SYNC})
- no-connect marks 0 -> 1
Other:
- moved on the sheet: U3
