File: _3_KICAD_BASE_BOARD/dspic33ak512mps512_baseboard/BLOCK_dsPIC33AK512MPS505.kicad_sch (KiCad schematic)
At the start: 19 parts, among them U2 dsPIC33AK512MPS505T-I/PT, Y1 ABMM-25.000MHZ-B2-T

Commit message: feat : 회로 작업중
Parts:
- C10, C11, C18: footprint (none) -> Capacitor_SMD:C_0603_1608Metric
- C12: renamed from C9; footprint (none) -> Capacitor_SMD:C_0603_1608Metric
- C13: renamed from C8; footprint (none) -> Capacitor_SMD:C_0603_1608Metric
- C14: renamed from C17; footprint (none) -> Capacitor_SMD:C_0603_1608Metric
- C15: renamed from C16; footprint (none) -> Capacitor_SMD:C_0603_1608Metric
- C16: renamed from C14; footprint (none) -> Capacitor_SMD:C_0603_1608Metric
- C17: renamed from C15; footprint (none) -> Capacitor_SMD:C_0603_1608Metric
- C19: renamed from C13; footprint (none) -> Capacitor_SMD:C_0603_1608Metric
- C20: renamed from C1; footprint (none) -> Capacitor_SMD:C_0603_1608Metric
- C21: renamed from C2; footprint (none) -> Capacitor_SMD:C_0603_1608Metric
- C9: renamed from C12; footprint (none) -> Capacitor_SMD:C_0603_1608Metric
- L1: value L_Small -> 10uH; footprint (none) -> Resistor_SMD:R_0603_1608Metric
- R1, R2, R3: footprint (none) -> Resistor_SMD:R_0603_1608Metric
- U1: renamed from U2; footprint TQFP48_PT_MCH -> dsPIC33AK512MPS505T-I/PT:TQFP48_PT_MCH
Connections:
- net CLK: now reaches U1.25 (RP39/SCL3/RC6)
- net MISO: now reaches U1.26 (RP40/SDA3/IOMAF7/RC7)
- net MOSI: now reaches U1.37 (RP49/PWM2H/IOMAD3/RD0)
- no-connect marks 15 -> 12
Other:
- moved on the sheet: C10, C11, C12, C13, C14, C15, C16, C17, C18, C19, C20, C21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
