File: _3_KICAD_BASE_BOARD/dspic33ak512mps512_baseboard/dspic33ak512mps512_baseboard.kicad_sch (KiCad schematic)
At the start: 0 parts

Commit message: feat : 회로 작업중
Other:
- sheet BLOCK_DIM_CONNECT ports: added COMM_BUS, DEBUG, DIM_BUS, I2C_BUS_0, SIGNAL_IO_BUS, SPI_BUS_0; removed none
- sheet BLOCK_SIGNAL_IO ports: added SIGNAL_IO_BUS, SPI_BUS_0; removed none
- sheet BLOCK_STROAGE ports: added I2C_BUS_0; removed none
- sheet BLOCK_TERMINAL ports: added COMM_BUS, DEBUG, DIM_BUS, SIGNAL_IO_BUS; removed none
- sheet BLOCK_dsPIC33AK512MPS505 ports: added COMM_BUS, DEBUG, I2C_BUS_0, SIGNAL_IO_BUS, SPI_BUS_0; removed none
