File: _3_KICAD_BOARD_2/kicad/BLOCK_DIM_CONNECT.kicad_sch (KiCad schematic)
At the start: 24 parts, among them J1 HTEC8-160-01-X-DV-A-BL-X

Commit message: feat : freerouting이 잘안됨..
Connections:
- net DIM_IO_20: no longer names the net of J1.31
- net DIM_IO_22: no longer names the net of J1.33
- net DIM_IO_24: no longer names the net of J1.35
- net DIM_IO_26: no longer names the net of J1.37
- net DIM_IO_28: no longer names the net of J1.39
Changed lines of the file:
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@@
 		)
 	)
-	(label "DIM_IO_26"
-		(at 71.12 115.57 0)
-		(effects
-			(font
-				(size 1.27 1.27)
-			)
-			(justify left bottom)
-		)
-	)
 	(label "DIM_IO_15"
 		(at 165.1 87.63 0)
@@
 		)
 	)
-	(label "{DIM_BUS}"
+	(label "DIM_BUS{DIM}"
 		(at 64.77 105.41 180)
 		(effects
@@
 		)
 	)
-	(label "DIM_IO_24"
-		(at 71.12 113.03 0)
-		(effects
-			(font
-				(size 1.27 1.27)
-			)
-			(justify left bottom)
-		)
-	)
 	(label "I2C_BUS.SCL"
 		(at 99.06 60.96 0)
@@
 		)
 	)
-	(label "DIM_IO_22"
-		(at 71.12 110.49 0)
-		(effects
-			(font
-				(size 1.27 1.27)
-			)
-			(justify left bottom)
-		)
-	)
 	(label "{DIM_BUS}"
 		(at 259.08 67.31 0)
@@
 		)
 	)
-	(label "DIM_IO_28"
-		(at 71.12 118.11 0)
-		(effects
-			(font
-				(size 1.27 1.27)
-			)
-			(justify left bottom)
-		)
-	)
 	(label "SIGNAL_IO_BUS.ADC_1_1"
 		(at 43.18 101.6 0)
@@
 		)
 	)
-	(label "DIM_IO_20"
-		(at 71.12 107.95 0)
-		(effects
-			(font
-				(size 1.27 1.27)
-			)
-			(justify left bottom)
-		)
-	)
 	(hierarchical_label "COMM_BUS"
 		(shape input)
@@
 		)
 		(instances
-			(project "dspic33ak512mps512_baseboard"
+			(project "kicad"
 				(path "/e24cf9e2-928b-48e3-96fe-45cdccce1592/e5eb7f35-5676-4c28-b984-cb300ec474a9"
 					(reference "#PWR06")
@@
 		)
 		(instances
-			(project "dspic33ak512mps512_baseboard"
+			(project "kicad"
 				(path "/e24cf9e2-928b-48e3-96fe-45cdccce1592/e5eb7f35-5676-4c28-b984-cb300ec474a9"
 					(reference "R6")
@@
 		)
 		(instances
-			(project "dspic33ak512mps512_baseboard"
+			(project "kicad"
 				(path "/e24cf9e2-928b-48e3-96fe-45cdccce1592/e5eb7f35-5676-4c28-b984-cb300ec474a9"
 					(reference "#PWR07")
@@
 		)
 		(instances
-			(project "dspic33ak512mps512_baseboard"
+			(project "kicad"
 				(path "/e24cf9e2-928b-48e3-96fe-45cdccce1592/e5eb7f35-5676-4c28-b984-cb300ec474a9"
 					(reference "R15")
@@
 		)
 		(instances
-			(project "dspic33ak512mps512_baseboard"
+			(project "kicad"
 				(path "/e24cf9e2-928b-48e3-96fe-45cdccce1592/e5eb7f35-5676-4c28-b984-cb300ec474a9"
 					(reference "R9")
@@
 		)
 		(instances
-			(project "dspic33ak512mps512_baseboard"
+			(project "kicad"
 				(path "/e24cf9e2-928b-48e3-96fe-45cdccce1592/e5eb7f35-5676-4c28-b984-cb300ec474a9"
 					(reference "#PWR09")
@@
 		)
 		(instances
-			(project "dspic33ak512mps512_baseboard"
+			(project "kicad"
 				(path "/e24cf9e2-928b-48e3-96fe-45cdccce1592/e5eb7f35-5676-4c28-b984-cb300ec474a9"
 					(reference "#PWR05")
@@
 		)
 		(instances
-			(project "dspic33ak512mps512_baseboard"
+			(project "kicad"
 				(path "/e24cf9e2-928b-48e3-96fe-45cdccce1592/e5eb7f35-5676-4c28-b984-cb300ec474a9"
 					(reference "C3")
@@
 		)
 		(instances
-			(project "dspic33ak512mps512_baseboard"
+			(project "kicad"
 				(path "/e24cf9e2-928b-48e3-96fe-45cdccce1592/e5eb7f35-5676-4c28-b984-cb300ec474a9"
 					(reference "R13")
@@
 		)
 		(instances
-			(project "dspic33ak512mps512_baseboard"
+			(project "kicad"
 				(path "/e24cf9e2-928b-48e3-96fe-45cdccce1592/e5eb7f35-5676-4c28-b984-cb300ec474a9"
 					(reference "C1")
@@
 		)
 		(instances
-			(project "dspic33ak512mps512_baseboard"
+			(project "kicad"
 				(path "/e24cf9e2-928b-48e3-96fe-45cdccce1592/e5eb7f35-5676-4c28-b984-cb300ec474a9"
 					(reference "#PWR011")
@@
 		)
 		(instances
-			(project "dspic33ak512mps512_baseboard"
+			(project "kicad"
 				(path "/e24cf9e2-928b-48e3-96fe-45cdccce1592/e5eb7f35-5676-4c28-b984-cb300ec474a9"
 					(reference "R10")
@@
 		)
 		(instances
-			(project "dspic33ak512mps512_baseboard"
+			(project "kicad"
 				(path "/e24cf9e2-928b-48e3-96fe-45cdccce1592/e5eb7f35-5676-4c28-b984-cb300ec474a9"
 					(reference "C6")
@@
 		)
 		(instances
-			(project "dspic33ak512mps512_baseboard"
+			(project "kicad"
 				(path "/e24cf9e2-928b-48e3-96fe-45cdccce1592/e5eb7f35-5676-4c28-b984-cb300ec474a9"
 					(reference "#PWR01")
@@
 		)
 		(instances
-			(project "dspic33ak512mps512_baseboard"
+			(project "kicad"
 				(path "/e24cf9e2-928b-48e3-96fe-45cdccce1592/e5eb7f35-5676-4c28-b984-cb300ec474a9"
 					(reference "R4")
@@
 		)
 		(instances
-			(project "dspic33ak512mps512_baseboard"
+			(project "kicad"
 				(path "/e24cf9e2-928b-48e3-96fe-45cdccce1592/e5eb7f35-5676-4c28-b984-cb300ec474a9"
 					(reference "#PWR03")
@@
 		)
 		(instances
-			(project "dspic33ak512mps512_baseboard"
+			(project "kicad"
 				(path "/e24cf9e2-928b-48e3-96fe-45cdccce1592/e5eb7f35-5676-4c28-b984-cb300ec474a9"
 					(reference "J1")
@@
 		)
 		(instances
-			(project "dspic33ak512mps512_baseboard"
+			(project "kicad"
 				(path "/e24cf9e2-928b-48e3-96fe-45cdccce1592/e5eb7f35-5676-4c28-b984-cb300ec474a9"
 					(reference "C7")
@@
 		)
 		(instances
-			(project "dspic33ak512mps512_baseboard"
+			(project "kicad"
 				(path "/e24cf9e2-928b-48e3-96fe-45cdccce1592/e5eb7f35-5676-4c28-b984-cb300ec474a9"
 					(reference "C8")
@@
 		)
 		(instances
-			(project "dspic33ak512mps512_baseboard"
+			(project "kicad"
 				(path "/e24cf9e2-928b-48e3-96fe-45cdccce1592/e5eb7f35-5676-4c28-b984-cb300ec474a9"
 					(reference "C5")
@@
 		)
 		(instances
-			(project "dspic33ak512mps512_baseboard"
+			(project "kicad"
 				(path "/e24cf9e2-928b-48e3-96fe-45cdccce1592/e5eb7f35-5676-4c28-b984-cb300ec474a9"
 					(reference "#PWR010")
@@
 		)
 		(instances
-			(project "dspic33ak512mps512_baseboard"
+			(project "kicad"
 				(path "/e24cf9e2-928b-48e3-96fe-45cdccce1592/e5eb7f35-5676-4c28-b984-cb300ec474a9"
 					(reference "R11")
@@
 		)
 		(instances
-			(project "dspic33ak512mps512_baseboard"
+			(project "kicad"
 				(path "/e24cf9e2-928b-48e3-96fe-45cdccce1592/e5eb7f35-5676-4c28-b984-cb300ec474a9"
 					(reference "R5")
@@
 		)
 		(instances
-			(project "dspic33ak512mps512_baseboard"
+			(project "kicad"
 				(path "/e24cf9e2-928b-48e3-96fe-45cdccce1592/e5eb7f35-5676-4c28-b984-cb300ec474a9"
 					(reference "R3")
@@
 		)
 		(instances
-			(project "dspic33ak512mps512_baseboard"
+			(project "kicad"
 				(path "/e24cf9e2-928b-48e3-96fe-45cdccce1592/e5eb7f35-5676-4c28-b984-cb300ec474a9"
 					(reference "J1")
@@
 		)
 		(instances
-			(project "dspic33ak512mps512_baseboard"
+			(project "kicad"
 				(path "/e24cf9e2-928b-48e3-96fe-45cdccce1592/e5eb7f35-5676-4c28-b984-cb300ec474a9"
 					(reference "R12")
@@
 		)
 		(instances
-			(project "dspic33ak512mps512_baseboard"
+			(project "kicad"
 				(path "/e24cf9e2-928b-48e3-96fe-45cdccce1592/e5eb7f35-5676-4c28-b984-cb300ec474a9"
 					(reference "#PWR012")
@@
 		)
 		(instances
-			(project "dspic33ak512mps512_baseboard"
+			(project "kicad"
 				(path "/e24cf9e2-928b-48e3-96fe-45cdccce1592/e5eb7f35-5676-4c28-b984-cb300ec474a9"
 					(reference "C2")
@@
 		)
 		(instances
-			(project "dspic33ak512mps512_baseboard"
+			(project "kicad"
 				(path "/e24cf9e2-928b-48e3-96fe-45cdccce1592/e5eb7f35-5676-4c28-b984-cb300ec474a9"
 					(reference "#PWR02")
@@
 		)
 		(instances
-			(project "dspic33ak512mps512_baseboard"
+			(project "kicad"
 				(path "/e24cf9e2-928b-48e3-96fe-45cdccce1592/e5eb7f35-5676-4c28-b984-cb300ec474a9"
 					(reference "#PWR04")
@@
 		)
 		(instances
-			(project "dspic33ak512mps512_baseboard"
+			(project "kicad"
 				(path "/e24cf9e2-928b-48e3-96fe-45cdccce1592/e5eb7f35-5676-4c28-b984-cb300ec474a9"
 					(reference "R7")
@@
 		)
 		(instances
-			(project "dspic33ak512mps512_baseboard"
+			(project "kicad"
 				(path "/e24cf9e2-928b-48e3-96fe-45cdccce1592/e5eb7f35-5676-4c28-b984-cb300ec474a9"
 					(reference "C4")
@@
 		)
 		(instances
-			(project "dspic33ak512mps512_baseboard"
+			(project "kicad"
 				(path "/e24cf9e2-928b-48e3-96fe-45cdccce1592/e5eb7f35-5676-4c28-b984-cb300ec474a9"
 					(reference "R14")
@@
 		)
 		(instances
-			(project "dspic33ak512mps512_baseboard"
+			(project "kicad"
 				(path "/e24cf9e2-928b-48e3-96fe-45cdccce1592/e5eb7f35-5676-4c28-b984-cb300ec474a9"
 					(reference "R8")
@@
 		)
 		(instances
-			(project "dspic33ak512mps512_baseboard"
+			(project "kicad"
 				(path "/e24cf9e2-928b-48e3-96fe-45cdccce1592/e5eb7f35-5676-4c28-b984-cb300ec474a9"
 					(reference "#PWR08")
@@
 		)
 		(instances
-			(project "dspic33ak512mps512_baseboard"
+			(project "kicad"
 				(path "/e24cf9e2-928b-48e3-96fe-45cdccce1592/e5eb7f35-5676-4c28-b984-cb300ec474a9"
 					(reference "R2")
@@
 		)
 		(instances
-			(project "dspic33ak512mps512_baseboard"
+			(project "kicad"
 				(path "/e24cf9e2-928b-48e3-96fe-45cdccce1592/e5eb7f35-5676-4c28-b984-cb300ec474a9"
 					(reference "R1")
