File: _6_KICAD_BOARD_DIM_ONLY/dspic33ak512/SIGNAL_IO_SHEET.kicad_sch (KiCad schematic)
At the start: 5 parts, among them U3 DAC7564ICPW

Commit message: feat : dim only project done
Parts:
- C26: renamed from C18; LCSC Part # (none) -> C14663
- C27: renamed from C19; LCSC Part # (none) -> C14663
- C28: renamed from C20; LCSC Part # (none) -> C14663
- R17: renamed from R1; LCSC Part # (none) -> C105588
- U3: LCSC Part # (none) -> C52451
Other:
- moved on the sheet: C26, C27, C28, R17, U3
