File: _6_KICAD_BOARD_DIM_ONLY/dspic33ak512/PWR_SHEET.kicad_sch (KiCad schematic)
At the start: 5 parts, among them U1 AZ1117H-3.3TRE1

Commit message: feat : dim board base board 작업시작
Parts:
- C3: LCSC Part # C602037 -> C86295
Changed lines of the file:
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@@
 			)
 		)
-		(property "LCSC Part #" "C602037"
+		(property "LCSC Part #" "C86295"
 			(at 165.1 92.71 0)
 			(effects
