File: _6_KICAD_BOARD_DIM_ONLY/dspic33ak512/STORAGE_SHEET.kicad_sch (KiCad schematic)
At the start: 4 parts, among them U4 FM24W256G

Commit message: feat : dim board base board 작업시작
Parts:
- R18, R19: LCSC Part # C114762 -> C4190
Changed lines of the file:
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@@
 			)
 		)
-		(property "LCSC Part #" "C114762"
+		(property "LCSC Part #" "C4190"
 			(at 160.02 81.28 0)
 			(effects
@@
 			)
 		)
-		(property "LCSC Part #" "C114762"
+		(property "LCSC Part #" "C4190"
 			(at 149.86 81.28 0)
 			(effects
